File: _autosave-apr.kicad_sch (KiCad schematic)
At the start: 94 parts, among them J1 Screw_Terminal_01x03, J10 Screw_Terminal_01x02, J11 Screw_Terminal_01x02, J12 Screw_Terminal_01x02, J13 Conn_01x04, J14 Conn_01x04, J15 Flash Module Conn, J16 Bateria Lítio 1, J17 Bateria Lítio 2, J18 LORA, J19 LORA, J2 Screw_Terminal_01x03, J20 Screw_Terminal_01x02, J21 Screw_Terminal_01x02, J22 Screw_Terminal_01x02, J23 Conn_01x20_Pin, J24 Conn_01x20_Pin, J25 Screw_Terminal_01x02, J26 Screw_Terminal_01x02, J27 Screw_Terminal_01x02, J28 Screw_Terminal_01x02, J29 A1, J3 Screw_Terminal_01x02, J30 Screw_Terminal_01x03, J31 Bateria Lítio 3, J32 Buzzer, J33 Bateria Lipo, J34 A2, J35 11, J36 12, J37 14, J4 Screw_Terminal_01x02, J5 Screw_Terminal_01x02, J6 Conn_01x20_Pin, J7 Conn_01x20_Pin, J8 Screw_Terminal_01x02, J9 Screw_Terminal_01x02, Q10 IRLZ34N, Q11 IRLZ34N, Q2 IRLZ34N, Q3 IRLZ34N, Q4 IRLZ34N, Q5 IRLZ34N, Q6 IRLZ34N, Q7 IRLZ34N, Q8 IRLZ34N, Q9 IRLZ34N, U3 LM7905_TO220

Commit message: Esquemático finalizado, Inicio do layout
Parts:
- J25, J27, J28: footprint TerminalBlock:TerminalBlock_bornier-2_P5.08mm -> Library:Screw Terminal 3D
Changed lines of the file:
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@@
 			)
 		)
-		(property "Footprint" "TerminalBlock:TerminalBlock_bornier-2_P5.08mm"
+		(property "Footprint" "Library:Screw Terminal 3D"
 			(at 452.12 114.3 0)
 			(effects
@@
 			)
 		)
-		(property "Footprint" "TerminalBlock:TerminalBlock_bornier-2_P5.08mm"
+		(property "Footprint" "Library:Screw Terminal 3D"
 			(at 452.12 138.43 0)
 			(effects
@@
 			)
 		)
-		(property "Footprint" "TerminalBlock:TerminalBlock_bornier-2_P5.08mm"
+		(property "Footprint" "Library:Screw Terminal 3D"
 			(at 452.12 90.17 0)
 			(effects
