File: apr.kicad_pcb (KiCad board)
At the start: 2 copper layers, 122.5 x 116.7 mm, 46 parts, among them J1 EMATCH, J10 Screw_Terminal_01x02, J11 Screw_Terminal_01x02, J18 LORA, J2 BATERIA, J3 Screw_Terminal_01x02, J4 Screw_Terminal_01x02, J5 Screw_Terminal_01x02, J6 Conn_01x20_Pin, J7 Conn_01x20_Pin, J8 Screw_Terminal_01x02, J9 Screw_Terminal_01x02, Q1 TIP120, Q10 TIP120, Q11 TIP120, Q2 TIP120, Q3 TIP120, Q4 TIP120, Q5 TIP120, Q6 TIP120, Q8 TIP120

Commit message: Revisão e ajustes
Parts:
- added D9: 1N4001, Diode_THT:D_DO-41_SOD81_P10.16mm_Horizontal, F.Cu at (116.7, 118.5)
- J18: footprint Connector_PinHeader_2.54mm:PinHeader_1x07_P2.54mm_Vertical -> Connector_PinSocket_2.54mm:PinSocket_1x07_P2.54mm_Vertical
- J6, J7: footprint Connector_PinHeader_2.54mm:PinHeader_1x20_P2.54mm_Vertical -> Connector_PinSocket_2.54mm:PinSocket_1x20_P2.54mm_Vertical
- moved D8 13.4 mm to (51.5, 42.4), turned to -90 degrees
- moved D6 9.04 mm to (52.0, 113.1), turned to 90 degrees
- moved D3 5.54 mm to (83.9, 118.5)
- moved D4 4.00 mm to (89.4, 41.7)
- moved D2 3.00 mm to (73.9, 41.7)
- moved D7 1.72 mm to (51.5, 76.6)
Connections:
- D1 pad 1: /VENT_PA1 -> +12V
- D1 pad 2: GND -> /VENT_PA1
- D2 pad 1: /INJECAO_PA7 -> +12V
- D2 pad 2: GND -> /INJECAO_PA7
- D3 pad 1: /LINHA_ABASTECE -> +12V
- D3 pad 2: GND -> /LINHA_ABASTECE
- D4 pad 1: /PURGA_TANQUE_PB0 -> +12V
- D4 pad 2: GND -> /PURGA_TANQUE_PB0
- D5 pad 1: /SUPERCHARGE_PA3 -> +12V
- D5 pad 2: GND -> /SUPERCHARGE_PA3
- D6 pad 1: /PURGA_LINHA_PA2 -> +12V
- D6 pad 2: GND -> /PURGA_LINHA_PA2
- D7 pad 1: /QUICK_DISCONNECT_PA4 -> +12V
- D7 pad 2: GND -> /QUICK_DISCONNECT_PA4
- D8 pad 1: /EMATCH -> +12V
- D8 pad 2: GND -> /EMATCH
- J6 pad 10: /ARM -> /QUICK
- J6 pad 11: /QUICK -> /SUPER
- J6 pad 12: /SUPER -> /PURGALINHA
- J6 pad 13: /PURGALINHA -> /VENT
- J6 pad 14: /VENT -> /LINHA
- J6 pad 15: /LINHA -> unconnected-(J6-Pin_15-Pad15)
- J6 pad 19: unconnected-(J6-Pin_19-Pad19) -> GND
- J6 pad 2: GND -> unconnected-(J6-Pin_2-Pad2)
- J6 pad 6: unconnected-(J6-Pin_6-Pad6) -> /PURGATANQUE
- J6 pad 7: /PURGATANQUE -> /INJECAO
- J6 pad 8: /INJECAO -> /IGNITE
- J6 pad 9: /IGNITE -> /ARM
Routing:
- net +12V: track 235.3 -> 337.0 mm
- net GND: track 15.2 -> 0.00 mm
- net /EMATCH: track 43.6 -> 32.8 mm
- net /PURGA_TANQUE_PB0: track 15.8 -> 24.1 mm
- net /INJECAO_PA7: track 15.0 -> 22.1 mm
- net Net-(Q1-E): track 68.6 -> 61.5 mm
- net /QUICK_DISCONNECT_PA4: track 24.2 -> 29.5 mm
- net /SUPERCHARGE_PA3: track 22.4 -> 27.5 mm
- net /LINHA_ABASTECE: track 21.2 -> 25.4 mm
- net /VENT_PA1: track 25.3 -> 29.3 mm
- net /LINHA: track 36.3 -> 32.7 mm
- net /PURGALINHA: track 34.4 -> 37.5 mm
- net /VENT: track 38.2 -> 41.2 mm
- net /SUPER: track 31.5 -> 33.7 mm
- net /PURGA_LINHA_PA2: track 22.7 -> 20.8 mm
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
Commit message: Ajustes finais
Parts:
- removed D9: 1N4001, Diode_THT:D_DO-41_SOD81_P10.16mm_Horizontal
Routing:
- net +12V: track 337.0 -> 324.0 mm
- net GND: track 0.00 -> 5.41 mm
Other:
- board text added: "+"

Commit message: Atualizações do dia 29_03
Parts:
- removed D4, D5, D6, D7: 1N4001, Diode_THT:D_DO-41_SOD81_P10.16mm_Horizontal
- removed J1: EMATCH, TerminalBlock:TerminalBlock_MaiXu_MX126-5.0-02P_1x02_P5.00mm
- removed J2: BATERIA, TerminalBlock:TerminalBlock_MaiXu_MX126-5.0-02P_1x02_P5.00mm
- removed Q1, Q2, Q3, Q4, Q5, Q6, Q8: TIP120, Package_TO_SOT_THT:TO-220-3_Vertical
- added D11: 1N4007, Diode_THT:D_DO-41_SOD81_P10.16mm_Horizontal, F.Cu at (217.2, 97.9)
- added D12: 1N4007, Diode_THT:D_DO-41_SOD81_P10.16mm_Horizontal, F.Cu at (217.2, 102.2)
- added D13: 1N4007, Diode_THT:D_DO-41_SOD81_P10.16mm_Horizontal, F.Cu at (217.2, 106.4)
- added D14: 1N4007, Diode_THT:D_DO-41_SOD81_P10.16mm_Horizontal, F.Cu at (217.2, 110.7)
- added D15: 1N4007, Diode_THT:D_DO-41_SOD81_P10.16mm_Horizontal, F.Cu at (217.2, 114.9)
- added D16: 1N4007, Diode_THT:D_DO-41_SOD81_P10.16mm_Horizontal, F.Cu at (217.2, 119.2)
- added D9: 1N4007, Diode_THT:D_DO-41_SOD81_P10.16mm_Horizontal, F.Cu at (217.2, 93.7)
- added J12: Screw_Terminal_01x02, TerminalBlock:TerminalBlock_MaiXu_MX126-5.0-02P_1x02_P5.00mm, F.Cu at (231.9, 57.7)
- added J13: Conn_01x04, TerminalBlock:TerminalBlock_MaiXu_MX126-5.0-04P_1x04_P5.00mm, F.Cu at (155.0, 157.6)
- added J14: Conn_01x04, TerminalBlock:TerminalBlock_MaiXu_MX126-5.0-04P_1x04_P5.00mm, F.Cu at (131.5, 175.6)
- added J15: Screw_Terminal_01x02, TerminalBlock:TerminalBlock_MaiXu_MX126-5.0-02P_1x02_P5.00mm, F.Cu at (231.9, 67.8)
- added J16: Screw_Terminal_01x02, TerminalBlock:TerminalBlock_MaiXu_MX126-5.0-02P_1x02_P5.00mm, F.Cu at (231.9, 78.0)
- added J17: Screw_Terminal_01x02, TerminalBlock:TerminalBlock_MaiXu_MX126-5.0-02P_1x02_P5.00mm, F.Cu at (244.4, 37.5)
- added J19: LORA, Connector_PinSocket_2.54mm:PinSocket_1x07_P2.54mm_Vertical, F.Cu at (258.7, 85.4)
- added J20: Screw_Terminal_01x02, TerminalBlock:TerminalBlock_MaiXu_MX126-5.0-02P_1x02_P5.00mm, F.Cu at (244.4, 47.6)
- added J21: Screw_Terminal_01x02, TerminalBlock:TerminalBlock_MaiXu_MX126-5.0-02P_1x02_P5.00mm, F.Cu at (244.4, 57.7)
- added J22: Screw_Terminal_01x02, TerminalBlock:TerminalBlock_MaiXu_MX126-5.0-02P_1x02_P5.00mm, F.Cu at (244.4, 67.8)
- added J23: Conn_01x20_Pin, Connector_PinSocket_2.54mm:PinSocket_1x20_P2.54mm_Vertical, F.Cu at (208.4, 34.8)
- added J24: Conn_01x20_Pin, Connector_PinSocket_2.54mm:PinSocket_1x20_P2.54mm_Vertical, F.Cu at (213.0, 34.8)
- added J25: Screw_Terminal_01x02, TerminalBlock:TerminalBlock_MaiXu_MX126-5.0-02P_1x02_P5.00mm, F.Cu at (29.3, 31.5)
- added J26: Screw_Terminal_01x02, TerminalBlock:TerminalBlock_MaiXu_MX126-5.0-02P_1x02_P5.00mm, F.Cu at (257.0, 37.5)
- added J27: Screw_Terminal_01x02, TerminalBlock:TerminalBlock_MaiXu_MX126-5.0-02P_1x02_P5.00mm, F.Cu at (257.0, 47.6)
- added J28: Screw_Terminal_01x02, TerminalBlock:TerminalBlock_MaiXu_MX126-5.0-02P_1x02_P5.00mm, F.Cu at (257.0, 57.7)
- added J29: Screw_Terminal_01x02, TerminalBlock:TerminalBlock_MaiXu_MX126-5.0-02P_1x02_P5.00mm, F.Cu at (257.0, 67.8)
- added Q12: TIP41, Package_TO_SOT_THT:TO-220-3_Vertical, F.Cu at (188.6, 54.3)
- added Q13: TIP41, Package_TO_SOT_THT:TO-220-3_Vertical, F.Cu at (188.6, 60.2)
- added Q14: TIP41, Package_TO_SOT_THT:TO-220-3_Vertical, F.Cu at (188.6, 66.2)
- added Q15: TIP41, Package_TO_SOT_THT:TO-220-3_Vertical, F.Cu at (188.6, 72.2)
- added Q16: TIP41, Package_TO_SOT_THT:TO-220-3_Vertical, F.Cu at (188.6, 78.1)
- added Q17: TIP41, Package_TO_SOT_THT:TO-220-3_Vertical, F.Cu at (188.6, 84.1)
- added Q18: TIP41, Package_TO_SOT_THT:TO-220-3_Vertical, F.Cu at (188.6, 90.0)
- added Q9: TIP41, Package_TO_SOT_THT:TO-220-3_Horizontal_TabDown, F.Cu at (70.0, 35.5)
- added R12: 100k, Resistor_THT:R_Axial_DIN0207_L6.3mm_D2.5mm_P15.24mm_Horizontal, F.Cu at (168.6, 79.0)
- added R13: 10k, Resistor_THT:R_Axial_DIN0207_L6.3mm_D2.5mm_P15.24mm_Horizontal, F.Cu at (168.6, 83.1)
- added R16: 5.6k, Resistor_THT:R_Axial_DIN0207_L6.3mm_D2.5mm_P15.24mm_Horizontal, F.Cu at (168.6, 95.2)
- added R17: 270k, Resistor_THT:R_Axial_DIN0207_L6.3mm_D2.5mm_P15.24mm_Horizontal, F.Cu at (168.6, 99.3)
- added R22: 390k, Resistor_THT:R_Axial_DIN0207_L6.3mm_D2.5mm_P15.24mm_Horizontal, F.Cu at (168.6, 119.5)
- added R23: 470, Resistor_THT:R_Axial_DIN0207_L6.3mm_D2.5mm_P15.24mm_Horizontal, F.Cu at (168.6, 123.6)
- added R24: 470, Resistor_THT:R_Axial_DIN0207_L6.3mm_D2.5mm_P15.24mm_Horizontal, F.Cu at (168.6, 127.6)
- added U3: LM7905_TO220, Package_TO_SOT_THT:TO-220-3_Vertical, F.Cu at (188.6, 96.0)
- D1, D8: value 1N4001 -> 1N4007
- D2, D3: value 1N4001 -> LED; footprint Diode_THT:D_DO-41_SOD81_P10.16mm_Horizontal -> LED_THT:LED_D5.0mm
- Q10, Q11: value TIP120 -> TIP41
- moved J10 187.2 mm to (231.9, 37.5), turned to 0 degrees
- moved J4 184.6 mm to (219.3, 47.6), turned to 0 degrees
- moved J5 180.1 mm to (219.3, 57.7), turned to 0 degrees
- moved D8 172.2 mm to (217.2, 89.4), turned to 0 degrees
- moved D2 170.7 mm to (231.7, 107.0)
- moved J11 169.6 mm to (231.9, 47.6)
- moved J8 149.3 mm to (219.3, 67.8)
- moved D1 148.3 mm to (217.2, 85.2), turned to 0 degrees
- moved D3 147.8 mm to (231.7, 114.5)
- moved J9 137.6 mm to (219.3, 78.0)
- moved J18 113.6 mm to (254.1, 85.4), turned to 0 degrees
- moved Q10 110.7 mm to (188.6, 42.4), turned to 0 degrees
- moved R20 110.1 mm to (168.6, 111.4)
- moved R6 105.8 mm to (168.6, 54.7)
- moved R18 103.7 mm to (168.6, 103.3)
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Connections:
- net /PURGA_TANQUE_PB0 renamed /PURGE_TANK
- D1 pad 2: /VENT_PA1 -> /IGNITE
- D2 pad 1: +12V -> Net-(D2-K)
- D2 pad 2: /INJECAO_PA7 -> +5V
- D3 pad 1: +12V -> Net-(D3-K)
- D3 pad 2: /LINHA_ABASTECE -> +3V3
- D8 pad 2: /EMATCH -> /SUPER_CHARGE
- J10 pad 2: /VENT_PA1 -> /VENT
- J11 pad 2: /LINHA_ABASTECE -> /FUEL_LINE
- J18 pad 1: /M0 -> /M0_PA11
- J18 pad 2: /M1 -> /M1_PA12
- J18 pad 3: /RX -> /TX1_PA9
- J18 pad 4: /TX -> /RX1_PA10
- J18 pad 5: unconnected-(J18-Pin_5-Pad5) -> /AUX_PB10
- J18 pad 6: +3V3 -> +5V
- J3 pad 2: /PURGA_LINHA_PA2 -> /PURGE_LINE
- J4 pad 2: /SUPERCHARGE_PA3 -> /SUPER_CHARGE
- J5 pad 2: /QUICK_DISCONNECT_PA4 -> /QUICK_DISCONNECT
- J6 pad 10: /QUICK -> /ARM_PA5
- J6 pad 11: /SUPER -> /QUICK_DISCONNECT_PA4
- J6 pad 12: /PURGALINHA -> /SUPER_CHARGE_PA3
- J6 pad 13: /VENT -> /PURGE_LINE_PA2
- J6 pad 14: /LINHA -> /VENT_PA1
- J6 pad 15: unconnected-(J6-Pin_15-Pad15) -> /FUEL_LINE_A0
- J6 pad 19: GND -> unconnected-(J6-Pin_19-Pad19)
- J6 pad 2: unconnected-(J6-Pin_2-Pad2) -> GND
- J6 pad 4: unconnected-(J6-Pin_4-Pad4) -> /AUX_PB10
- J6 pad 5: unconnected-(J6-Pin_5-Pad5) -> /RESET_PB2
- J6 pad 6: /PURGATANQUE -> /SAVE_PB1
- J6 pad 7: /INJECAO -> /PURGE_TANK_PB0
- J6 pad 8: /IGNITE -> /INJECTION_PA7
- J6 pad 9: /ARM -> /IGNITE_PA6
- J7 pad 12: unconnected-(J7-Pin_12-Pad12) -> /M1_PA12
- J7 pad 13: unconnected-(J7-Pin_13-Pad13) -> /M0_PA11
- J7 pad 14: /RX -> /RX1_PA10
- J7 pad 15: /TX -> /TX1_PA9
- J7 pad 16: /M1 -> unconnected-(J7-Pin_16-Pad16)
- J7 pad 17: /M0 -> unconnected-(J7-Pin_17-Pad17)
- J7 pad 3: unconnected-(J7-Pin_3-Pad3) -> +5V
- J8 pad 2: /INJECAO_PA7 -> /INJECTION
- Q10 pad 2: /INJECAO_PA7 -> /INJECTION
- R1 pad 1: /ARM -> /ARM_PA5
- R10 pad 2: /SUPER -> /SUPER_CHARGE_PA3
- R11 pad 1: /SUPER -> /SUPER_CHARGE_PA3
- R14 pad 2: /QUICK -> /QUICK_DISCONNECT_PA4
- R15 pad 1: /QUICK -> /QUICK_DISCONNECT_PA4
- R18 pad 2: /INJECAO -> /INJECTION_PA7
- R19 pad 1: /INJECAO -> /INJECTION_PA7
- R2 pad 1: /IGNITE -> /IGNITE_PA6
- R20 pad 2: /PURGATANQUE -> /PURGE_TANK_PB0
- R21 pad 1: /PURGATANQUE -> /PURGE_TANK_PB0
- R3 pad 2: /IGNITE -> /IGNITE_PA6
- R4 pad 2: /LINHA -> /FUEL_LINE_A0
- R5 pad 1: /LINHA -> /FUEL_LINE_A0
- R6 pad 2: /VENT -> /VENT_PA1
- R7 pad 1: /VENT -> /VENT_PA1
- R8 pad 2: /PURGALINHA -> /PURGE_LINE_PA2
- R9 pad 1: /PURGALINHA -> /PURGE_LINE_PA2
Routing:
- net +12V: track 324.0 -> 0.00 mm
- net Net-(Q1-E): track 61.5 -> 0.00 mm
- net /TX: track 55.4 -> 0.00 mm
- net /VENT: track 41.2 -> 0.00 mm
- net /PURGALINHA: track 37.5 -> 0.00 mm
- net Net-(Q18-B): track 36.2 -> 0.00 mm
- net Net-(Q16-B): track 34.5 -> 0.00 mm
- net Net-(Q17-B): track 33.8 -> 0.00 mm
- net /SUPER: track 33.7 -> 0.00 mm
- net /EMATCH: track 32.8 -> 0.00 mm
- net /LINHA: track 32.7 -> 0.00 mm
- net +3V3: track 32.5 -> 0.00 mm
- net Net-(Q15-B): track 32.2 -> 0.00 mm
- net Net-(Q9-B): track 31.8 -> 0.00 mm
- net /QUICK: track 30.3 -> 0.00 mm
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- removed copper zone on B.Cu, net GND
Other:
- board outline removed
- board text removed: "+"
- board text removed: "12V"
- board text removed: "EMATCH"
- board text removed: "INJECAO"
- board text removed: "LINHA"
- board text removed: "M0"
- board text removed: "M1"
- board text removed: "PLACA DE ATUACAO - PROJETO JUPITER"
- board text removed: "PURGALINHA"
- board text removed: "PURGATANQUE"
- board text removed: "QUICK"
- board text removed: "RX"
- board text removed: "SUPERCHARGE"
- board text removed: "TX"
- board text removed: "VENT"

Commit message: Esquemático finalizado, Inicio do layout
Parts:
- removed D11, D12, D13, D14, D15, D16, D8, D9: 1N4007, Diode_THT:D_DO-41_SOD81_P10.16mm_Horizontal
- removed Q12, Q13, Q14, Q15, Q16, Q17, Q18: TIP41, Package_TO_SOT_THT:TO-220-3_Vertical
- removed R10, R12, R3, R4, R6, R8: 100k, Resistor_THT:R_Axial_DIN0207_L6.3mm_D2.5mm_P15.24mm_Horizontal
- removed R11, R13, R5, R7, R9: 10k, Resistor_THT:R_Axial_DIN0207_L6.3mm_D2.5mm_P15.24mm_Horizontal
- added C1: 1uF, Capacitor_THT:CP_Radial_D4.0mm_P1.50mm, B.Cu at (82.6, 102.1)
- added CR1: UF4007-E3/73, Diode_THT:D_DO-15_P15.24mm_Horizontal, B.Cu at (157.2, 108.2)
- added CR2: UF4007-E3/73, Diode_THT:D_DO-15_P15.24mm_Horizontal, B.Cu at (157.4, 78.3)
- added CR3: UF4007-E3/73, Diode_THT:D_DO-15_P15.24mm_Horizontal, B.Cu at (79.3, 152.4)
- added CR4: UF4007-E3/73, Diode_THT:D_DO-15_P15.24mm_Horizontal, B.Cu at (157.2, 90.9)
- added CR5: UF4007-E3/73, Diode_THT:D_DO-15_P15.24mm_Horizontal, B.Cu at (133.8, 67.3)
- added CR6: UF4007-E3/73, Diode_THT:D_DO-15_P15.24mm_Horizontal, B.Cu at (90.9, 67.0)
- added CR7: UF4007-E3/73, Diode_THT:D_DO-15_P15.24mm_Horizontal, B.Cu at (138.7, 146.8)
- added CR8: UF4007-E3/73, Diode_THT:D_DO-15_P15.24mm_Horizontal, B.Cu at (157.1, 119.0)
- added D10: LED, LED_THT:LED_D3.0mm, B.Cu at (143.6, 124.3)
- added D17: LED, LED_THT:LED_D3.0mm, B.Cu at (148.2, 138.7)
- added D18: LED, LED_THT:LED_D3.0mm, B.Cu at (112.1, 71.1)
- added D19: LED, LED_THT:LED_D3.0mm, B.Cu at (69.8, 116.3)
- added D20: LED, LED_THT:LED_D3.0mm, B.Cu at (148.7, 100.5)
- added D4: 1N4007, Diode_THT:D_DO-41_SOD81_P10.16mm_Horizontal, B.Cu at (157.5, 127.3)
- added D5: LED, LED_THT:LED_D3.0mm, B.Cu at (146.6, 71.0)
- added D6: LED, LED_THT:LED_D3.0mm, B.Cu at (148.6, 84.8)
- added D7: LED, LED_THT:LED_D3.0mm, B.Cu at (111.2, 60.9)
- added J1: Screw_Terminal_01x03, Library:KT100-3PIN, F.Cu at (105.8, 49.2)
- added J2: Screw_Terminal_01x03, Library:KT100-3PIN, F.Cu at (141.8, 48.5)
- added J30: Screw_Terminal_01x03, Library:KT100-3PIN, F.Cu at (176.7, 48.1)
- added J31: Bateria Lítio 3, Library:Screw Terminal 3D, B.Cu at (222.7, 155.5)
- added J32: Buzzer, TerminalBlock:TerminalBlock_bornier-2_P5.08mm, B.Cu at (180.2, 157.7)
- added J33: Bateria Lipo, Library:Screw Terminal 3D, B.Cu at (77.9, 86.5)
- added J34: A2, Connector_PinHeader_2.54mm:PinHeader_1x01_P2.54mm_Vertical, B.Cu at (181.4, 143.9)
- added J35: 11, Connector_PinHeader_2.54mm:PinHeader_1x01_P2.54mm_Vertical, B.Cu at (168.8, 143.8)
- added J36: 12, Connector_PinHeader_2.54mm:PinHeader_1x01_P2.54mm_Vertical, B.Cu at (181.3, 131.8)
- added J37: 14, Connector_PinHeader_2.54mm:PinHeader_1x01_P2.54mm_Vertical, B.Cu at (169.0, 131.8)
- added Q2: IRLZ34N, Package_TO_SOT_THT:TO-220-3_Vertical, B.Cu at (122.9, 111.0)
- added Q3: IRLZ34N, Package_TO_SOT_THT:TO-220-3_Vertical, B.Cu at (123.0, 88.7)
- added Q4: IRLZ34N, Package_TO_SOT_THT:TO-220-3_Vertical, B.Cu at (123.0, 99.5)
- added Q5: IRLZ34N, Package_TO_SOT_THT:TO-220-3_Vertical, B.Cu at (92.5, 146.4)
- added Q6: IRLZ34N, Package_TO_SOT_THT:TO-220-3_Vertical, B.Cu at (123.2, 147.1)
- added Q7: IRLZ34N, Package_TO_SOT_THT:TO-220-3_Vertical, B.Cu at (123.0, 122.5)
- added Q8: IRLZ34N, Package_TO_SOT_THT:TO-220-3_Vertical, B.Cu at (122.8, 76.3)
- added R25: 2k, Resistor_SMD:R_0805_2012Metric, F.Cu at (162.3, 71.7)
- added R26: 470, Resistor_SMD:R_0805_2012Metric, F.Cu at (106.4, 61.4)
- added R27: 470, Resistor_SMD:R_0805_2012Metric, F.Cu at (139.5, 124.4)
- added R28: 470, Resistor_SMD:R_0805_2012Metric, F.Cu at (141.7, 138.4)
- added R29: 470, Resistor_SMD:R_0805_2012Metric, F.Cu at (103.2, 72.2)
- added R30: 470, Resistor_SMD:R_0805_2012Metric, F.Cu at (71.0, 122.2)
- added R31: 470, Resistor_SMD:R_0805_2012Metric, F.Cu at (143.1, 100.5)
- added R32: 4K7, Resistor_SMD:R_0805_2012Metric, F.Cu at (95.0, 143.3)
- added R33: 4K7, Resistor_SMD:R_0805_2012Metric, F.Cu at (124.2, 143.4)
- added R34: 4K7, Resistor_SMD:R_0805_2012Metric, F.Cu at (166.7, 71.8)
- added R35: 4K7, Resistor_SMD:R_0805_2012Metric, F.Cu at (125.6, 130.7)
- added U1: ~, Library:hx711, B.Cu at (219.5, 80.5)
- added U2: ~, Library:hx711, B.Cu at (219.3, 102.7)
- D1, D2, D3, J18, J19, J23, J24, J6, J7, U3: moved to B.Cu
- J10, J11, J12, J20, J21, J22, J26, J3, J4, J5, J8, J9: footprint TerminalBlock:TerminalBlock_MaiXu_MX126-5.0-02P_1x02_P5.00mm -> TerminalBlock:TerminalBlock_bornier-2_P5.08mm; moved to B.Cu
- J13, J14: footprint TerminalBlock:TerminalBlock_MaiXu_MX126-5.0-04P_1x04_P5.00mm -> TerminalBlock:TerminalBlock_bornier-4_P5.08mm; moved to B.Cu
- J15: value Screw_Terminal_01x02 -> Flash Module Conn; footprint TerminalBlock:TerminalBlock_MaiXu_MX126-5.0-02P_1x02_P5.00mm -> Connector_PinSocket_2.54mm:PinSocket_1x06_P2.54mm_Vertical; moved to B.Cu
- J16: value Screw_Terminal_01x02 -> Bateria Lítio 1; footprint TerminalBlock:TerminalBlock_MaiXu_MX126-5.0-02P_1x02_P5.00mm -> Library:Screw Terminal 3D; moved to B.Cu
- J17: value Screw_Terminal_01x02 -> Bateria Lítio 2; footprint TerminalBlock:TerminalBlock_MaiXu_MX126-5.0-02P_1x02_P5.00mm -> Library:Screw Terminal 3D; moved to B.Cu
- J25, J27, J28: footprint TerminalBlock:TerminalBlock_MaiXu_MX126-5.0-02P_1x02_P5.00mm -> Library:Screw Terminal 3D; moved to B.Cu
- J29: value Screw_Terminal_01x02 -> A1; footprint TerminalBlock:TerminalBlock_MaiXu_MX126-5.0-02P_1x02_P5.00mm -> Connector_PinHeader_2.54mm:PinHeader_1x01_P2.54mm_Vertical; moved to B.Cu
- Q10, Q11: value TIP41 -> IRLZ34N; moved to B.Cu
- Q9: value TIP41 -> IRLZ34N; footprint Package_TO_SOT_THT:TO-220-3_Horizontal_TabDown -> Package_TO_SOT_THT:TO-220-3_Vertical; moved to B.Cu
- R1, R15: value 10k -> 470; footprint Resistor_THT:R_Axial_DIN0207_L6.3mm_D2.5mm_P15.24mm_Horizontal -> Resistor_SMD:R_0805_2012Metric
- R14, R18, R20: value 100k -> 4K7; footprint Resistor_THT:R_Axial_DIN0207_L6.3mm_D2.5mm_P15.24mm_Horizontal -> Resistor_SMD:R_0805_2012Metric
- R16, R17, R2, R22, R23, R24: footprint Resistor_THT:R_Axial_DIN0207_L6.3mm_D2.5mm_P15.24mm_Horizontal -> Resistor_SMD:R_0805_2012Metric
- R19, R21: value 10k -> 4K7; footprint Resistor_THT:R_Axial_DIN0207_L6.3mm_D2.5mm_P15.24mm_Horizontal -> Resistor_SMD:R_0805_2012Metric
- moved J25 239.5 mm to (233.8, 156.1), turned to 0 degrees
- moved J3 206.1 mm to (239.4, 67.6), turned to -90 degrees
- moved J26 192.8 mm to (106.6, 158.1)
- moved J11 183.1 mm to (70.6, 134.2), turned to 90 degrees
- moved J18 180.7 mm to (79.5, 131.8)
- moved J27 180.1 mm to (78.2, 68.8), turned to 90 degrees
- moved J28 179.2 mm to (78.4, 42.9), turned to -90 degrees
- moved J9 165.5 mm to (71.0, 151.2), turned to 90 degrees
- moved J5 162.0 mm to (92.2, 158.1), turned to 180 degrees
- moved R2 145.6 mm to (218.8, 124.4), turned to -90 degrees
- moved J10 143.5 mm to (88.7, 27.7)
- moved J6 138.9 mm to (105.8, 136.8)
- moved J14 135.1 mm to (240.2, 95.4), turned to 90 degrees
- moved J12 131.1 mm to (147.5, 158.1), turned to 180 degrees
- moved J21 128.0 mm to (164.5, 157.7), turned to 180 degrees
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Connections:
- D1 pad 1: +12V -> +12C
- J10 pad 1: +12V -> +12C
- J11 pad 1: +12V -> +12L
- J15 pad 1: /TRANSDUCER_CAMARA_I+ -> +3V3
- J15 pad 2: /TRANSDUCER_CAMARA_I- -> /FLASH_CS
- J16 pad 1: /TRANSDUCER_TANK_I+ -> GND
- J16 pad 2: /TRANSDUCER_TANK_I- -> +12C
- J17 pad 1: /TRANSDUCER_LINE_I+ -> GND
- J17 pad 2: /TRANSDUCER_LINE_I- -> +12L
- J23 pad 11: /MISO_PA15 -> /FLASH_MISO
- J23 pad 12: /MOSI_PA12 -> /FLASH_MOSI
- J23 pad 13: /SCK_PA11 -> /FLASH_SCK
- J23 pad 16: /CS_PA8 -> /FLASH_CS
- J23 pad 19: /M1_B13 -> /M1_PB13
- J23 pad 20: /M0_B12 -> /M0_PB12
- J24 pad 16: /RESET_PB2 -> /RESET_PB3
- J26 pad 1: +12V -> +12C
- J29 pad 1: GND -> +12V
- J3 pad 1: +12V -> +12L
- J4 pad 1: +12V -> +12L
- J5 pad 1: +12V -> +12C
- J6 pad 5: /RESET_PB2 -> unconnected-(J6-Pin_5-Pad5)
- J7 pad 10: unconnected-(J7-Pin_10-Pad10) -> /RESET_PB3
- J8 pad 1: +12V -> +12L
- J9 pad 1: +12V -> +12L
- Q10 pad 1: Net-(Q10-B) -> /IGNITE_PA6
- Q10 pad 2: /INJECTION -> /IGNITE
- Q11 pad 1: Net-(Q11-B) -> Net-(Q11-G)
- Q11 pad 2: /PURGE_TANK -> Net-(D4-A)
- Q9 pad 1: Net-(Q9-B) -> /FUEL_LINE_A0
- Q9 pad 2: /QUICK_DISCONNECT -> /FUEL_LINE
- R1 pad 1: /ARM_PA5 -> Net-(D5-K)
- R1 pad 2: Net-(Q17-B) -> /PURGE_LINE
- R15 pad 1: /QUICK_DISCONNECT_PA4 -> Net-(D6-K)
- R15 pad 2: Net-(Q9-B) -> /PURGE_LINE
- R18 pad 2: /INJECTION_PA7 -> /PURGE_LINE_PA2
- R19 pad 1: /INJECTION_PA7 -> GND
- R19 pad 2: Net-(Q10-B) -> /SUPER_CHARGE_PA3
- R2 pad 1: /IGNITE_PA6 -> /FLASH_CS
- R20 pad 2: /PURGE_TANK_PB0 -> /VENT_PA1
- R21 pad 1: /PURGE_TANK_PB0 -> GND
- R21 pad 2: Net-(Q11-B) -> /FUEL_LINE_A0
- U3 pad 2: Net-(J29-Pin_2) -> Net-(J33-Pin_1)
Routing:
- net +12C: track 0.00 -> 215.5 mm
- net /FUEL_LINE: track 0.00 -> 196.6 mm
- net /IGNITE: track 0.00 -> 179.3 mm
- net +12V: track 0.00 -> 141.9 mm
- net +5V: track 0.00 -> 120.8 mm, vias 0 -> 2
- net /TRANSDUCER_LINE_PA2: track 0.00 -> 114.9 mm, vias 0 -> 2
- net /THERMISTOR_CAMARA: track 0.00 -> 114.7 mm
- net /QUICK_DISCONNECT: track 0.00 -> 112.9 mm, vias 0 -> 2
- net /THERMISTOR_LINE: track 0.00 -> 105.1 mm
- net /ARM_PA5: track 0.00 -> 97.9 mm
- net /TRANSDUCER_TANK_PA1: track 0.00 -> 93.3 mm
- net +12L: track 0.00 -> 92.0 mm
- net /AUX_PB10: track 0.00 -> 79.3 mm, vias 0 -> 2
- net /INJECTION: track 0.00 -> 74.6 mm
- net +3V3: track 0.00 -> 74.4 mm
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- added copper zone on F.Cu, net GND
