File: apr.kicad_sch (KiCad schematic)
At the start: 94 parts, among them J1 Screw_Terminal_01x03, J10 Screw_Terminal_01x02, J11 Screw_Terminal_01x02, J12 Screw_Terminal_01x02, J13 Conn_01x04, J14 Conn_01x04, J15 Flash Module Conn, J16 Bateria Lítio 1, J17 Bateria Lítio 2, J18 LORA, J19 LORA, J2 Screw_Terminal_01x03, J20 Screw_Terminal_01x02, J21 Screw_Terminal_01x02, J22 Screw_Terminal_01x02, J23 Conn_01x20_Pin, J24 Conn_01x20_Pin, J25 Screw_Terminal_01x02, J26 Screw_Terminal_01x02, J27 Screw_Terminal_01x02, J28 Screw_Terminal_01x02, J29 A1, J3 Screw_Terminal_01x02, J30 Screw_Terminal_01x03, J31 Bateria Lítio 3, J32 Buzzer, J33 Bateria Lipo, J34 A2, J35 11, J36 12, J37 14, J4 Screw_Terminal_01x02, J5 Screw_Terminal_01x02, J6 Conn_01x20_Pin, J7 Conn_01x20_Pin, J8 Screw_Terminal_01x02, J9 Screw_Terminal_01x02, Q10 IRLZ34N, Q11 IRLZ34N, Q2 IRLZ34N, Q3 IRLZ34N, Q4 IRLZ34N, Q5 IRLZ34N, Q6 IRLZ34N, Q7 IRLZ34N, Q8 IRLZ34N, Q9 IRLZ34N, U3 LM7905_TO220

Commit message: Versão 1.0 placa híbrido - 1 camada
Parts:
- D10, D17, D18, D19, D20, D5, D6, D7: footprint LED_THT:LED_D3.0mm -> LED_THT:LED_D5.0mm
- J25, J27, J28: footprint TerminalBlock:TerminalBlock_bornier-2_P5.08mm -> Library:Screw Terminal 3D
Changed lines of the file:
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@@
 			)
 		)
-		(property "Footprint" "LED_THT:LED_D3.0mm"
+		(property "Footprint" "LED_THT:LED_D5.0mm"
 			(at 102.87 299.72 0)
 			(effects
@@
 			)
 		)
-		(property "Footprint" "TerminalBlock:TerminalBlock_bornier-2_P5.08mm"
+		(property "Footprint" "Library:Screw Terminal 3D"
 			(at 452.12 114.3 0)
 			(effects
@@
 			)
 		)
-		(property "Footprint" "LED_THT:LED_D3.0mm"
+		(property "Footprint" "LED_THT:LED_D5.0mm"
 			(at 99.06 367.03 0)
 			(effects
@@
 			)
 		)
-		(property "Footprint" "LED_THT:LED_D3.0mm"
+		(property "Footprint" "LED_THT:LED_D5.0mm"
 			(at 102.87 236.22 0)
 			(effects
@@
 			)
 		)
-		(property "Footprint" "TerminalBlock:TerminalBlock_bornier-2_P5.08mm"
+		(property "Footprint" "Library:Screw Terminal 3D"
 			(at 452.12 138.43 0)
 			(effects
@@
 			)
 		)
-		(property "Footprint" "LED_THT:LED_D3.0mm"
+		(property "Footprint" "LED_THT:LED_D5.0mm"
 			(at 204.47 365.76 0)
 			(effects
@@
 			)
 		)
-		(property "Footprint" "LED_THT:LED_D3.0mm"
+		(property "Footprint" "LED_THT:LED_D5.0mm"
 			(at 102.87 176.53 0)
 			(effects
@@
 			)
 		)
-		(property "Footprint" "TerminalBlock:TerminalBlock_bornier-2_P5.08mm"
+		(property "Footprint" "Library:Screw Terminal 3D"
 			(at 452.12 90.17 0)
 			(effects
@@
 			)
 		)
-		(property "Footprint" "LED_THT:LED_D3.0mm"
+		(property "Footprint" "LED_THT:LED_D5.0mm"
 			(at 203.2 238.76 0)
 			(effects
@@
 			)
 		)
-		(property "Footprint" "LED_THT:LED_D3.0mm"
+		(property "Footprint" "LED_THT:LED_D5.0mm"
 			(at 203.2 302.26 0)
 			(effects
@@
 			)
 		)
-		(property "Footprint" "LED_THT:LED_D3.0mm"
+		(property "Footprint" "LED_THT:LED_D5.0mm"
 			(at 203.2 173.99 0)
 			(effects

Commit message: Esquemático e Layout PCB Sólido
Parts:
- removed CR2, CR3, CR4, CR5, CR6, CR7, CR8: UF4007-E3/73, Diode_THT:D_DO-15_P15.24mm_Horizontal, symbol Diode UF4007:UF4007-E3_73
- removed D1: 1N4007, Diode_THT:D_DO-41_SOD81_P10.16mm_Horizontal, symbol Diode:1N4007
- removed D10, D17, D18, D19, D2, D20, D3: LED, LED_THT:LED_D5.0mm, symbol Device:LED
- removed J1, J2: Screw_Terminal_01x03, Library:KT100-3PIN, symbol Connector:Screw_Terminal_01x03
- removed J10, J11, J12, J20, J21, J22, J3, J4, J5, J8, J9: Screw_Terminal_01x02, TerminalBlock:TerminalBlock_bornier-2_P5.08mm, symbol Connector:Screw_Terminal_01x02
- removed J14: Conn_01x04, TerminalBlock:TerminalBlock_bornier-4_P5.08mm, symbol Connector_Generic:Conn_01x04
- removed J16: Bateria Lítio 1, Library:Screw Terminal 3D, symbol Connector:Screw_Terminal_01x02
- removed J17: Bateria Lítio 2, Library:Screw Terminal 3D, symbol Connector:Screw_Terminal_01x02
- removed J27, J28: Screw_Terminal_01x02, Library:Screw Terminal 3D, symbol Connector:Screw_Terminal_01x02
- removed J29: A1, Connector_PinHeader_2.54mm:PinHeader_1x01_P2.54mm_Vertical, symbol Connector:Conn_01x01_Pin
- removed J34: A2, Connector_PinHeader_2.54mm:PinHeader_1x01_P2.54mm_Vertical, symbol Connector:Conn_01x01_Pin
- removed J35: 11, Connector_PinHeader_2.54mm:PinHeader_1x01_P2.54mm_Vertical, symbol Connector:Conn_01x01_Pin
- removed J36: 12, Connector_PinHeader_2.54mm:PinHeader_1x01_P2.54mm_Vertical, symbol Connector:Conn_01x01_Pin
- removed J37: 14, Connector_PinHeader_2.54mm:PinHeader_1x01_P2.54mm_Vertical, symbol Connector:Conn_01x01_Pin
- removed Q2, Q3, Q4, Q5, Q6, Q7, Q8, Q9: IRLZ34N, Package_TO_SOT_THT:TO-220-3_Vertical, symbol Transistor_FET:IRLZ34N
- removed R1, R15, R23, R24, R29, R30, R31: 470, Resistor_SMD:R_0805_2012Metric, symbol Device:R
- removed R14, R18, R19, R20, R21, R32, R33, R34: 4K7, Resistor_SMD:R_0805_2012Metric, symbol Device:R
- removed R16: 5.6k, Resistor_SMD:R_0805_2012Metric, symbol Device:R
- removed R17: 270k, Resistor_SMD:R_0805_2012Metric, symbol Device:R
- removed R22: 390k, Resistor_SMD:R_0805_2012Metric, symbol Device:R
- removed U1: ~, Library:hx711, symbol Library:HX711
- added K1: Fujitsu_FTR-LYCA005x, Relay_THT:Relay_SPDT_Finder_36.11, symbol Relay:Fujitsu_FTR-LYCA005x
- added U1: Ag9905LP, Converter_DCDC:Converter_DCDC_Silvertel_Ag99xxLP_THT, symbol Converter_DCDC:Ag9905LP
- CR1: footprint Diode_THT:D_DO-15_P15.24mm_Horizontal -> Diode_THT:D_A-405_P12.70mm_Horizontal
- J25: value Screw_Terminal_01x02 -> VSUPPLY TRANSDUCER
- J26: value Screw_Terminal_01x02 -> IGNITION; footprint TerminalBlock:TerminalBlock_bornier-2_P5.08mm -> Library:Screw Terminal 3D
- J31: value Bateria Lítio 3 -> Bateria Lítio
- J32: footprint TerminalBlock:TerminalBlock_bornier-2_P5.08mm -> Library:Screw Terminal 3D
Connections:
- net +12C is gone; now on net +12V: CR1.1, J26.1 (Pin_1)
- net ARM is gone; now on an unnamed net: R27.2
- net INJECTION is gone; now on an unnamed net: R28.2
- net QUICK_DISCONNECT is gone; now on net IGNITE: CR1.2
- net VENT is gone; now on an unnamed net: R26.2
- net +12V: now also K1.A1
- net +3.3V: now also D5.2 (A), J7.1 (Pin_1); no longer U2.7 (VDD)
- net +3V3: now also D7.2 (A), U2.7 (VDD); no longer J7.1 (Pin_1)
- net +5V: no longer D5.2 (A), D7.2 (A)
- net GND: now also R26.1, R27.1, R28.1, K1.11
- net at D4.2 (A), Q11.2 (D): now also K1.A2
- net at D7.1 (K): no longer R26.1
- net at J32.2 (Pin_2): now also K1.14
- net DT2: no longer names the net of J23.7 (Pin_7)
- net FUEL_LINE_A0: no longer names the net of J6.15 (Pin_15)
- net INJECTION_PA7: no longer names the net of J6.8 (Pin_8)
- net PURGE_LINE_PA2: no longer names the net of J6.13 (Pin_13)
- net PURGE_TANK_PB0: no longer names the net of J6.7 (Pin_7)
- net QUICK_DISCONNECT_PA4: no longer names the net of J6.11 (Pin_11)
- net SCK2: no longer names the net of J23.8 (Pin_8)
- net SUPER_CHARGE_PA3: no longer names the net of J6.12 (Pin_12)
- net THERMISTOR_CAMARA: no longer names the net of J24.10 (Pin_10)
- net THERMISTOR_LINE: no longer names the net of J24.11 (Pin_11)
- net THERMISTOR_TANK: no longer names the net of J24.12 (Pin_12)
- net TRANSDUCER_CAMARA_PA0 renamed TRANSDUCER
- net TRANSDUCER_LINE_PA2: no longer names the net of J24.13 (Pin_13)
- net TRANSDUCER_TANK_PA1: no longer names the net of J24.14 (Pin_14)
- net VENT_PA1: no longer names the net of J6.14 (Pin_14)
- new net: U1.1 (+VDC), U1.2 (+VDC)
- new net: U1.5 (VIN+), U1.6 (VIN+)
- new net: U1.7 (VIN-), U1.8 (VIN-)
- no-connect marks 40 -> 57
Other:
- note added: "LED ACTUADOR 3V3"
- note added: "LED TRANSMISSION 3V3"
- note added: "VSUPPLY 12V"
- note added: "VSUPPLY LED 5V"
- note removed: "A+2"
- note removed: "A-2"
- note removed: "ARM"
- note removed: "BATERIAS"
- note removed: "E+2"
- note removed: "E-2"
- note removed: "LOAD CELL 10 Hz"
- note removed: "THERMISTOR CAMARA"
- note removed: "THERMISTOR LINE"
- note removed: "THERMISTOR TANK"
- note removed: "VALVE: INJECTION"
- note removed: "VALVE: LINE"
- note removed: "VALVE: PURGE LINE"
- note removed: "VALVE: PURGE TANK"
- note removed: "VALVE: QUICK DISCONNECT"
- note removed: "VALVE: SUPERCHARGE"
- note removed: "VALVE: VENT"
- note removed: "VALVES"
- note removed: "VSUPPLY: AMPERE SENSOR 1"
- note removed: "VSUPPLY: AMPERE SENSOR 2"
- note removed: "VSUPPLY: PRESSURE TRANSDUCER LINE"
- note removed: "VSUPPLY: PRESSURE TRANSDUCER TANK"
- moved on the sheet: J25, J26, J30, J31

Commit message: Layout Final
Parts:
- removed Q11: IRLZ34N, Package_TO_SOT_THT:TO-220-3_Vertical, symbol Transistor_FET:IRLZ34N
- removed U1: Ag9905LP, Converter_DCDC:Converter_DCDC_Silvertel_Ag99xxLP_THT, symbol Converter_DCDC:Ag9905LP
- added CR2: UF4007-E3/73, Diode_THT:D_A-405_P12.70mm_Horizontal, symbol Diode UF4007:UF4007-E3_73
- added J27: ARM, Library:Screw Terminal 3D, symbol Connector:Screw_Terminal_01x02
- added Q1: BC547, Package_TO_SOT_THT:TO-92_Inline, symbol Transistor_BJT:BC547
- added Q12: IRLZ34N, Package_TO_SOT_THT:TO-220-3_Vertical, symbol Transistor_FET:IRLZ34N
- added R36: 4K7, Resistor_SMD:R_0805_2012Metric, symbol Device:R
Connections:
- net +12V: now also D5.2 (A), CR2.1, J27.1 (Pin_1)
- net +3.3V: no longer D5.2 (A)
- net +5V: now also J6.1 (Pin_1); no longer J7.3 (Pin_3)
- net GND: now also J24.10 (Pin_10), J24.11 (Pin_11), J24.12 (Pin_12), J24.13 (Pin_13), J24.14 (Pin_14), Q1.3 (E), Q12.3 (S), R36.1
- net at D4.2 (A), K1.A2: now also Q1.1 (C)
- net SAVE_PA1: now reaches J6.15 (Pin_15)
- net SAVE_PA1: now also J23.6 (Pin_6)
- net at R25.2: now also Q1.2 (B)
- net ARM_PA5 renamed ARM_PA6
- net ARM_PA6: now also J6.9 (Pin_9), Q12.1 (G), R36.2; no longer J6.10 (Pin_10)
- net IGNITE_PA6 renamed IGINTE_PA5
- net IGINTE_PA5: now also J6.10 (Pin_10); no longer J6.9 (Pin_9)
- net M0_PB12 renamed M0_PB13
- net M0_PB13: now also J23.19 (Pin_19); no longer J23.20 (Pin_20)
- net M1_PB13 renamed M1_PB12
- net M1_PB12: now also J23.20 (Pin_20); no longer J23.19 (Pin_19)
- net SAVE_PB1: no longer names the net of J6.6 (Pin_6)
- net SAVE_PB1: no longer J23.6 (Pin_6)
- new net ARM: CR2.2, J27.2 (Pin_2), Q12.2 (D)
- no-connect marks 57 -> 47
Other:
- note added: "ARM"
- note added: "LED HX"
- note added: "LED LITIUM BAT"
- note removed: "LED ACTUADOR 3V3"
- note removed: "LED TRANSMISSION 3V3"
- note removed: "VSUPPLY LED 5V"
- moved on the sheet: D5, D6, J13, J15, J18, J19, J23, J24, J25, J30, J31, J6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
